File: Configurable_PIR_GreenPak.kicad_sch (KiCad schematic)
At the start: 31 parts, among them SW1 SW_Push, SW2 SW_Push, SW3 SW_SPDT, U1 PIR, U2 SLG47001V

Commit message: Create basic PCB layout after assigning footprints to all schematic symbols
Parts:
- BT1: value CR2477 cell -> Battery_Cell; footprint (none) -> Configurable_PIR_GreenPAK:MPD_BU2477SM-JJ-GTR; PN BU2477SM-JJ-GTR -> (none)
- C1, C6, C8: footprint (none) -> Configurable_PIR_GreenPAK:C_0805_2012Metric; PN (none) -> CC0805MKX5R6BB226
- C2, C3, C4, C5, C7, C9: footprint (none) -> Configurable_PIR_GreenPAK:C_0402_1005Metric
- D1, D2: footprint (none) -> Configurable_PIR_GreenPAK:5990Kxx_reverse_LED
- D3: footprint (none) -> Configurable_PIR_GreenPAK:D_SOD-323
- H1, H2, H3, H4: footprint (none) -> Configurable_PIR_GreenPAK:MountingHole_3.2mm_M3
- R1, R2, R3, R4, R5, R6, R7, R8: footprint (none) -> Configurable_PIR_GreenPAK:R_0402_1005Metric
- SW1, SW2: footprint (none) -> Configurable_PIR_GreenPAK:RT3301AF100Q
- SW3: footprint (none) -> Configurable_PIR_GreenPAK:SW_500ASSP1SM6QE
- U1: footprint (none) -> Configurable_PIR_GreenPAK:TO-5-3
- U2: footprint (none) -> Configurable_PIR_GreenPAK:Renesas_UQFN-20_2x3mm_P0.4mm_LayoutBorder4x6y
Connections:
- net 1V4_REF: no longer U2.17 (GPIO2), U2.20 (GPIO3)
- net DOWN_BTN: no longer U2.15 (GPIO0)
- net ENABLE_SW: no longer U2.1 (GPI0)
- net GND: now also BT1.N; no longer BT1.2 (-), U2.3 (GND)
- net LOW_BAT_LED: no longer U2.19 (SDA/GPIO5)
- net PIR_LED: no longer U2.18 (SCL/GPIO4)
- net PIR_OUT: no longer U2.6 (OA0+)
- net STAGE1_OUT: now also U2.11 (OA1+); no longer C8.1, U2.8 (OA0_OUT)
- net STAGE2_OUT: no longer U2.9 (OA1_OUT)
- net UP_BTN: no longer U2.16 (GPIO1)
- net VBAT: now also BT1.P (+); no longer BT1.1 (+), U2.14 (VDDA), U2.2 (VDD)
- net VDD/2_REF: no longer U2.11 (OA1+)
- net at C7.1, D3.1 (K), R4.2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: no longer U2.7 (OA0-)
- net at C9.1, R6.1: no longer U2.10 (OA1-), U2.5 (RH0_B/GPI2)
- net at U2.12 (RH1_B/GPI3): no longer U2.4 (RH0_A/GPI1)
- net at U2.13 (RH1_A/GPI4): no longer C8.2
- new net: C8.1, U2.10 (OA1-)
